File: esp32_gsh_env_sensors.kicad_pcb (KiCad board)
At the start: 2 copper layers, 0 parts

Commit message: Setup PCB layout for JLCPCB manufacturing
Other:
- rule pad_to_mask_clearance: 0 -> 0.05
Changed lines of the file:
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@@
   )
   (setup
-    (pad_to_mask_clearance 0)
+    (stackup
+      (layer "F.SilkS" (type "Top Silk Screen") (color "White"))
+      (layer "F.Paste" (type "Top Solder Paste"))
+      (layer "F.Mask" (type "Top Solder Mask") (color "Black") (thickness 0.01))
+      (layer "F.Cu" (type "copper") (thickness 0.035))
+      (layer "dielectric 1" (type "prepreg") (thickness 1.51) (material "FR4") (epsilon_r 4.5) (loss_tangent 0.02))
+      (layer "B.Cu" (type "copper") (thickness 0.035))
+      (layer "B.Mask" (type "Bottom Solder Mask") (color "Black") (thickness 0.01))
+      (layer "B.Paste" (type "Bottom Solder Paste"))
+      (layer "B.SilkS" (type "Bottom Silk Screen") (color "White"))
+      (copper_finish "None")
+      (dielectric_constraints no)
+    )
+    (pad_to_mask_clearance 0.05)
+    (solder_mask_min_width 0.254)
+    (pad_to_paste_clearance_ratio -0.12)
     (pcbplotparams
       (layerselection 0x00010fc_ffffffff)
